File: hardware/DALI_CCT_48V_30W/DALI_CCT_48V_30W.kicad_pcb (KiCad board)
At the start: 4 copper layers, 150 x 60 mm, 8 parts, among them J1 48V_IN 5.08mm, J2 DALI 5.08mm, J3 LED 5.08mm, J4 SWD 1.27mm

Commit message: Schritt 3: KiCad Schaltplan und PCB-Layout ergänzt (OI-011/OI-012)
Co-authored-by: manuelh83 <208121220+manuelh83@users.noreply.github.com>
Parts:
- added Q_CW: STB20NF06L D2PAK 60V/20A Rth_jc=3.1°C/W, Package_TO_SOT_SMD:TO-263-3_TabDown, B.Cu at (115.0, 42.0)
- added Q_WW: STB20NF06L D2PAK 60V/20A Rth_jc=3.1°C/W, Package_TO_SOT_SMD:TO-263-3_TabDown, B.Cu at (100.0, 42.0)
Routing:
- net WW-: vias 0 -> 9
- net CW-: vias 0 -> 9
- added copper zone on B.Cu, net CW-
- added copper zone on B.Cu, net WW-
Other:
- board text added: "ISO BARRIER: CLR>=2mm / CRG>=5mm / ZONE=8mm (IEC 62368-1:2018, Reinf., PD2, OVC II, IIIa, 63V)"
- board text added: "Q_WW / Q_CW: STB20NF06L D2PAK (Rev A.1 - replaces SOT-223) 9 thermal vias 3x3 grid (0.3mm drill/0.5mm pad) under exposed tab 20x20mm B.Cu thermal pour per channel coupled to Al enclosure via TIM Rth(j-ambient) ~7.8C/W; Tj~64C at 50C ambient with adaptive bus voltage See design-specification.md §4.4 for full thermal calculation"
- board text removed: "DALI ISOLATION KEEPOUT ZONE (8mm min, no copper/vias)"
Changed lines of the file:
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@@
     (effects (font (size 0.8 0.8)) (justify center))
   )
-  (gr_text "DALI ISOLATION KEEPOUT ZONE (8mm min, no copper/vias)"
+  (gr_text "ISO BARRIER: CLR>=2mm / CRG>=5mm / ZONE=8mm\n(IEC 62368-1:2018, Reinf., PD2, OVC II, IIIa, 63V)"
     (at 28 30 90)
     (layer "Cmts.User")
@@
     (effects (font (size 1.2 1.2)) (justify center))
   )
+  (footprint "Package_TO_SOT_SMD:TO-263-3_TabDown"
+    (layer "B.Cu")
+    (at 100 42)
+    (descr "D2PAK STB20NF06L - Rev A.1 replaces SOT-223 for thermal improvement")
+    (attr smd)
+    (property "Reference" "Q_WW" (at 100 36 0) (layer "B.SilkS") (effects (font (size 1.27 1.27))))
+    (property "Value" "STB20NF06L D2PAK 60V/20A Rth_jc=3.1°C/W" (at 100 50 0) (layer "B.Fab") (effects (font (size 1.0 1.0))))
+    (property "MPN" "STMicro STB20NF06L" (at 0 0 0) (layer "B.Fab") (effects (font (size 0.5 0.5)) (hide yes)))
+    (fp_line (start 94.8 40.4) (end 105.2 40.4) (layer "B.Fab") (width 0.12))
+    (fp_line (start 94.8 40.4) (end 94.8 49.5) (layer "B.Fab") (width 0.12))
+    (fp_line (start 105.2 49.5) (end 94.8 49.5) (layer "B.Fab") (width 0.12))
+    (fp_line (start 105.2 40.4) (end 105.2 49.5) (layer "B.Fab") (width 0.12))
+    (fp_line (start 94.8 40.4) (end 105.2 40.4) (layer "B.CrtYd") (width 0.05))
+    (fp_line (start 94.8 40.4) (end 94.8 49.5) (layer "B.CrtYd") (width 0.05))
+    (fp_line (start 105.2 49.5) (end 94.8 49.5) (layer "B.CrtYd") (width 0.05))
+    (fp_line (start 105.2 40.4) (end 105.2 49.5) (layer "B.CrtYd") (width 0.05))
+    (fp_text type user "9x THERMAL VIA 3x3 GRID" (at 100 46.826 0) (layer "B.SilkS") (effects (font (size 0.6 0.6)) (hide yes)))
+    (pad "1" smd rect (at 97.714 42.000 0) (size 1.7 2.4) (layers "B.Cu" "B.Paste" "B.Mask")
+      (net 0 "")
+    )
+    (pad "2" smd rect (at 100.000 42.000 0) (size 1.7 2.4) (layers "B.Cu" "B.Paste" "B.Mask")
+      (net 2 "PGND")
+    )
+    (pad "3" smd rect (at 100.000 46.826 0) (size 9.0 6.0) (layers "B.Cu" "B.Paste" "B.Mask")
+      (net 5 "WW-")
+    )
+  )
+  (via
+    (at 98.500 45.326)
+    (size 0.5)
+    (drill 0.3)
+    (layers "F.Cu" "B.Cu")
+    (net 5 "WW-")
+  )
+  (via
+    (at 98.500 46.826)
+    (size 0.5)
+    (drill 0.3)
+    (layers "F.Cu" "B.Cu")
+    (net 5 "WW-")
+  )
+  (via
+    (at 98.500 48.326)
+    (size 0.5)
+    (drill 0.3)
+    (layers "F.Cu" "B.Cu")
+    (net 5 "WW-")
+  )
+  (via
+    (at 100.000 45.326)
+    (size 0.5)
+    (drill 0.3)
+    (layers "F.Cu" "B.Cu")
+    (net 5 "WW-")
+  )
+  (via
+    (at 100.000 46.826)
+    (size 0.5)
+    (drill 0.3)
+    (layers "F.Cu" "B.Cu")
+    (net 5 "WW-")
+  )
+  (via
+    (at 100.000 48.326)
+    (size 0.5)
+    (drill 0.3)
+    (layers "F.Cu" "B.Cu")
+    (net 5 "WW-")
+  )
+  (via
+    (at 101.500 45.326)
+    (size 0.5)
+    (drill 0.3)
+    (layers "F.Cu" "B.Cu")
+    (net 5 "WW-")
+  )
+  (via
+    (at 101.500 46.826)
+    (size 0.5)
+    (drill 0.3)
+    (layers "F.Cu" "B.Cu")
+    (net 5 "WW-")
+  )
+  (via
+    (at 101.500 48.326)
+    (size 0.5)
+    (drill 0.3)
+    (layers "F.Cu" "B.Cu")
+    (net 5 "WW-")
+  )
+  (zone
+    (net 5 "WW-")
+    (layer "B.Cu")
+    (name "THERMAL_Q_WW")
+    (hatch edge 0.508)
+    (connect_pads (thermal_gap 0.5) (thermal_bridge_width 1.0))
+    (min_thickness 0.25)
+    (filled_areas_thickness yes)
+    (fill yes (thermal_gap 0.5) (thermal_bridge_width 1.0))
+    (polygon (pts (xy 90 36.826) (xy 110 36.826) (xy 110 56.826) (xy 90 56.826)))
+  )
+  (footprint "Package_TO_SOT_SMD:TO-263-3_TabDown"
+    (layer "B.Cu")
+    (at 115 42)
+    (descr "D2PAK STB20NF06L - Rev A.1 replaces SOT-223 for thermal improvement")
+    (attr smd)
+    (property "Reference" "Q_CW" (at 115 36 0) (layer "B.SilkS") (effects (font (size 1.27 1.27))))
+    (property "Value" "STB20NF06L D2PAK 60V/20A Rth_jc=3.1°C/W" (at 115 50 0) (layer "B.Fab") (effects (font (size 1.0 1.0))))
+    (property "MPN" "STMicro STB20NF06L" (at 0 0 0) (layer "B.Fab") (effects (font (size 0.5 0.5)) (hide yes)))
+    (fp_line (start 109.8 40.4) (end 120.2 40.4) (layer "B.Fab") (width 0.12))
+    (fp_line (start 109.8 40.4) (end 109.8 49.5) (layer "B.Fab") (width 0.12))
+    (fp_line (start 120.2 49.5) (end 109.8 49.5) (layer "B.Fab") (width 0.12))
+    (fp_line (start 120.2 40.4) (end 120.2 49.5) (layer "B.Fab") (width 0.12))
+    (fp_line (start 109.8 40.4) (end 120.2 40.4) (layer "B.CrtYd") (width 0.05))
+    (fp_line (start 109.8 40.4) (end 109.8 49.5) (layer "B.CrtYd") (width 0.05))
+    (fp_line (start 120.2 49.5) (end 109.8 49.5) (layer "B.CrtYd") (width 0.05))
+    (fp_line (start 120.2 40.4) (end 120.2 49.5) (layer "B.CrtYd") (width 0.05))
+    (fp_text type user "9x THERMAL VIA 3x3 GRID" (at 115 46.826 0) (layer "B.SilkS") (effects (font (size 0.6 0.6)) (hide yes)))
+    (pad "1" smd rect (at 112.714 42.000 0) (size 1.7 2.4) (layers "B.Cu" "B.Paste" "B.Mask")
+      (net 0 "")
+    )
+    (pad "2" smd rect (at 115.000 42.000 0) (size 1.7 2.4) (layers "B.Cu" "B.Paste" "B.Mask")
+      (net 2 "PGND")
+    )
+    (pad "3" smd rect (at 115.000 46.826 0) (size 9.0 6.0) (layers "B.Cu" "B.Paste" "B.Mask")
+      (net 6 "CW-")
+    )
+  )
+  (via
+    (at 113.500 45.326)
+    (size 0.5)
+    (drill 0.3)
+    (layers "F.Cu" "B.Cu")
+    (net 6 "CW-")
+  )
+  (via
+    (at 113.500 46.826)
+    (size 0.5)
+    (drill 0.3)
+    (layers "F.Cu" "B.Cu")
+    (net 6 "CW-")
+  )
+  (via
+    (at 113.500 48.326)
+    (size 0.5)
+    (drill 0.3)
+    (layers "F.Cu" "B.Cu")
+    (net 6 "CW-")
+  )
+  (via
+    (at 115.000 45.326)
+    (size 0.5)
+    (drill 0.3)
+    (layers "F.Cu" "B.Cu")
+    (net 6 "CW-")
+  )
+  (via
+    (at 115.000 46.826)
+    (size 0.5)
+    (drill 0.3)
+    (layers "F.Cu" "B.Cu")
+    (net 6 "CW-")
+  )
+  (via
+    (at 115.000 48.326)
+    (size 0.5)
+    (drill 0.3)
+    (layers "F.Cu" "B.Cu")
+    (net 6 "CW-")
+  )
+  (via
+    (at 116.500 45.326)
+    (size 0.5)
+    (drill 0.3)
+    (layers "F.Cu" "B.Cu")
+    (net 6 "CW-")
+  )
+  (via
+    (at 116.500 46.826)
+    (size 0.5)
+    (drill 0.3)
+    (layers "F.Cu" "B.Cu")
+    (net 6 "CW-")
+  )
+  (via
+    (at 116.500 48.326)
+    (size 0.5)
+    (drill 0.3)
+    (layers "F.Cu" "B.Cu")
+    (net 6 "CW-")
+  )
+  (zone
+    (net 6 "CW-")
+    (layer "B.Cu")
+    (name "THERMAL_Q_CW")
+    (hatch edge 0.508)
+    (connect_pads (thermal_gap 0.5) (thermal_bridge_width 1.0))
+    (min_thickness 0.25)
+    (filled_areas_thickness yes)
+    (fill yes (thermal_gap 0.5) (thermal_bridge_width 1.0))
+    (polygon (pts (xy 105 36.826) (xy 125 36.826) (xy 125 56.826) (xy 105 56.826)))
+  )
+  (gr_text "Q_WW / Q_CW: STB20NF06L D2PAK (Rev A.1 - replaces SOT-223)\n9 thermal vias 3x3 grid (0.3mm drill/0.5mm pad) under exposed tab\n20x20mm B.Cu thermal pour per channel coupled to Al enclosure via TIM\nRth(j-ambient) ~7.8C/W; Tj~64C at 50C ambient with adaptive bus voltage\nSee design-specification.md §4.4 for full thermal calculation"
+    (at 107 57 0)
+    (layer "Cmts.User")
+    (effects (font (size 0.7 0.7)) (justify center))
+  )
 )
